File: splanck throughhole.sch (KiCad schematic (older format))
At the start: 51 parts, among them K1 XLR3, SW1 SW_PUSH, SW10 SW_PUSH, SW11 SW_PUSH, SW12 SW_PUSH, SW13 SW_PUSH, SW14 SW_PUSH, SW15 SW_PUSH, SW16 SW_PUSH, SW17 SW_PUSH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

Commit message: Added a row to schematic
I'm really new to this, but adding this row didn't seem impossible :)
Parts:
- added D? (x6): D, cherry mx:DIODE, symbol D
- added SW13, SW14, SW21, SW25, SW5, SW9: SW_PUSH, cherry mx:CHERRY_PCB_100H, symbol SW_PUSH
- K1: symbol XLR3 -> XLR3-RESCUE-splanck_throughhole
- U1: symbol ATmega32U4-AU -> ATmega32U4-AU-RESCUE-splanck_throughhole
Connections:
- net labels added: row4
- wire segments 10 -> 11
Changed lines of the file:
@@
 EESchema Schematic File Version 2
+LIBS:splanck throughhole-rescue
 LIBS:power
 LIBS:device
@@
 Connection ~ 6550 4000
 Wire Wire Line
-	5250 2050 5250 3700
+	5250 2050 5250 4250
 Connection ~ 5250 2600
 Connection ~ 5250 3150
 Wire Wire Line
-	5950 2050 5950 3700
+	5950 2050 5950 4250
 Connection ~ 5950 2600
 Connection ~ 5950 3150
 Wire Wire Line
-	6700 2050 6700 3700
+	6700 2050 6700 4250
 Connection ~ 6700 3150
 Connection ~ 6700 2600
 Wire Wire Line
-	7400 2050 7400 3700
+	7400 2050 7400 4250
 Connection ~ 7400 2600
 Connection ~ 7400 3150
 Wire Wire Line
-	8100 2050 8100 3700
+	8100 2050 8100 4250
 Connection ~ 8100 3150
 Connection ~ 8100 2600
 Wire Wire Line
-	8800 2050 8800 3700
+	8800 2050 8800 4250
 Connection ~ 8800 2600
 Connection ~ 8800 3150
 $Comp
-L ATmega32U4-AU U1
+L ATmega32U4-AU-RESCUE-splanck_throughhole U1
 U 1 1 574B317C
 P 2450 3250
@@
 data
 $Comp
-L XLR3 K1
+L XLR3-RESCUE-splanck_throughhole K1
 U 1 1 574BAB3B
 P 5100 1250
@@
 	0    1    1    0
 $EndComp
+$Comp
+L SW_PUSH SW5
+U 1 1 5AB55323
+P 5550 4250
+F 0 "SW5" H 5700 4360 50  0000 C CNN
+F 1 "SW_PUSH" H 5550 4170 50  0000 C CNN
+F 2 "cherry mx:CHERRY_PCB_100H" H 5550 4250 50  0001 C CNN
+F 3 "" H 5550 4250 50  0000 C CNN
+	1    5550 4250
+	1    0    0    -1
+$EndComp
+$Comp
+L D D?
+U 1 1 5AB5552F
+P 5850 4400
+F 0 "D?" H 5850 4500 50  0000 C CNN
+F 1 "D" H 5850 4300 50  0000 C CNN
+F 2 "cherry mx:DIODE" H 5850 4400 50  0001 C CNN
+F 3 "" H 5850 4400 50  0000 C CNN
+	1    5850 4400
+	0    1    1    0
+$EndComp
+$Comp
+L SW_PUSH SW9
+U 1 1 5AB55604
+P 6250 4250
+F 0 "SW9" H 6400 4360 50  0000 C CNN
+F 1 "SW_PUSH" H 6250 4170 50  0000 C CNN
+F 2 "cherry mx:CHERRY_PCB_100H" H 6250 4250 50  0001 C CNN
+F 3 "" H 6250 4250 50  0000 C CNN
+	1    6250 4250
+	1    0    0    -1
+$EndComp
+$Comp
+L D D?
+U 1 1 5AB556CA
+P 6550 4400
+F 0 "D?" H 6550 4500 50  0000 C CNN
+F 1 "D" H 6550 4300 50  0000 C CNN
+F 2 "cherry mx:DIODE" H 6550 4400 50  0001 C CNN
+F 3 "" H 6550 4400 50  0000 C CNN
+	1    6550 4400
+	0    1    1    0
+$EndComp
+$Comp
+L SW_PUSH SW13
+U 1 1 5AB55797
+P 7000 4250
+F 0 "SW13" H 7150 4360 50  0000 C CNN
+F 1 "SW_PUSH" H 7000 4170 50  0000 C CNN
+F 2 "cherry mx:CHERRY_PCB_100H" H 7000 4250 50  0001 C CNN
+F 3 "" H 7000 4250 50  0000 C CNN
+	1    7000 4250
+	1    0    0    -1
+$EndComp
+$Comp
+L D D?
+U 1 1 5AB55861
+P 7300 4400
+F 0 "D?" H 7300 4500 50  0000 C CNN
+F 1 "D" H 7300 4300 50  0000 C CNN
+F 2 "cherry mx:DIODE" H 7300 4400 50  0001 C CNN
+F 3 "" H 7300 4400 50  0000 C CNN
+	1    7300 4400
+	0    1    1    0
+$EndComp
+$Comp
+L SW_PUSH SW14
+U 1 1 5AB5596B
+P 7700 4250
+F 0 "SW14" H 7850 4360 50  0000 C CNN
+F 1 "SW_PUSH" H 7700 4170 50  0000 C CNN
+F 2 "cherry mx:CHERRY_PCB_100H" H 7700 4250 50  0001 C CNN
+F 3 "" H 7700 4250 50  0000 C CNN
+	1    7700 4250
+	1    0    0    -1
+$EndComp
+$Comp
+L D D?
+U 1 1 5AB55A3B
+P 8000 4400
+F 0 "D?" H 8000 4500 50  0000 C CNN
+F 1 "D" H 8000 4300 50  0000 C CNN
+F 2 "cherry mx:DIODE" H 8000 4400 50  0001 C CNN
+F 3 "" H 8000 4400 50  0000 C CNN
+	1    8000 4400
+	0    1    1    0
+$EndComp
+$Comp
+L SW_PUSH SW21
+U 1 1 5AB55B12
+P 8400 4250
+F 0 "SW21" H 8550 4360 50  0000 C CNN
+F 1 "SW_PUSH" H 8400 4170 50  0000 C CNN
+F 2 "cherry mx:CHERRY_PCB_100H" H 8400 4250 50  0001 C CNN
+F 3 "" H 8400 4250 50  0000 C CNN
+	1    8400 4250
+	1    0    0    -1
+$EndComp
+$Comp
+L D D?
+U 1 1 5AB55BEA
+P 8700 4400
+F 0 "D?" H 8700 4500 50  0000 C CNN
+F 1 "D" H 8700 4300 50  0000 C CNN
+F 2 "cherry mx:DIODE" H 8700 4400 50  0001 C CNN
+F 3 "" H 8700 4400 50  0000 C CNN
+	1    8700 4400
+	0    1    1    0
+$EndComp
+$Comp
+L SW_PUSH SW25
+U 1 1 5AB55E5D
+P 9100 4250
+F 0 "SW25" H 9250 4360 50  0000 C CNN
+F 1 "SW_PUSH" H 9100 4170 50  0000 C CNN
+F 2 "cherry mx:CHERRY_PCB_100H" H 9100 4250 50  0001 C CNN
+F 3 "" H 9100 4250 50  0000 C CNN
+	1    9100 4250
+	1    0    0    -1
+$EndComp
+$Comp
+L D D?
+U 1 1 5AB55F39
+P 9400 4400
+F 0 "D?" H 9400 4500 50  0000 C CNN
+F 1 "D" H 9400 4300 50  0000 C CNN
+F 2 "cherry mx:DIODE" H 9400 4400 50  0001 C CNN
+F 3 "" H 9400 4400 50  0000 C CNN
+	1    9400 4400
+	0    1    1    0
+$EndComp
+Connection ~ 5250 3700
+Connection ~ 5950 3700
+Connection ~ 6700 3700
+Connection ~ 7400 3700
+Connection ~ 8100 3700
+Connection ~ 8800 3700
+Wire Wire Line
+	5850 4550 9400 4550
+Connection ~ 6550 4550
+Connection ~ 7300 4550
+Connection ~ 8000 4550
+Connection ~ 8700 4550
+Text GLabel 5850 4550 0    60   Input ~ 0
+row4
 $EndSCHEMATC
